Commit message: fixed world, added colour to robot, uncommented section in C code

File: src/my_robot/urdf/my_robot.xacro (robot description, xacro)
@@ -2,4 +2,13 @@
 <robot name="my_robot" xmlns:xacro="http://www.ros.org/wiki/xacro">
   <xacro:include filename="$(find my_robot)/urdf/my_robot.gazebo" />
+  <gazebo reference="chassis">
+     <material>Gazebo/Green</material>
+  </gazebo>
+  <gazebo reference="left_wheel">
+     <material>Gazebo/Red</material>
+  </gazebo>
+  <gazebo reference="right_wheel">
+     <material>Gazebo/Blue</material>
+  </gazebo>
   <link name="robot_footprint"></link>
   <joint name="robot_footprint_joint" type="fixed">
